File: ATOM_CAN_BOARD_RJ45_v0.1/M5Atom_CAN_RJ45.sch (KiCad schematic (older format))
At the start: 9 parts, among them J1 RJ45, J2 RJ45, J3 Conn_01x06_Male, J4 Conn_01x02_Male, U1 MCP2562-E-P, U2 ATOM_Lite

Commit message: ATOM_CAN_BOARD_v0.2 and RJ45_v0.1 update
Parts:
- added D1: D_Schottky, Diode_SMD:D_TUMD2, symbol Device:D_Schottky
- U2: symbol M5:ATOM_Lite -> M5Atom_CAN_RJ45-rescue:ATOM_Lite-M5
Connections:
- net +5V: now also D1.2 (A); no longer C2.1, U1.3 (VDD), U2.3 (+5V)
- new net: C2.1, D1.1 (K), U1.3 (VDD), U2.3 (+5V)
Other:
- moved on the sheet: C1, C2, J1, J2, J3, J4, R1, U1, U2
